File: hardware/nrf52840_sensor_hub.kicad_sch (KiCad schematic)
At the start: 8 parts, among them J1 FTSH-105-01-L-DV, J2 TYPE-C-16P-01, J3 B2B-PH-SM4-TB, U1 Raytac MDBT50Q-1M, U2 BME280, U3 LSM6DSO, U4 MCP73831T-2ACI/OT, U5 TPS7A2033PDBVR

Commit message: fix: resolve KiCad 8/9 S-expression symbol unit naming in schematic
Parts:
- J1: symbol Sensor_Hub:SWD_Header_10Pin -> SWD_Header_10Pin
- J2: symbol Sensor_Hub:USB_C_Receptacle_16P -> USB_C_Receptacle_16P
- J3: symbol Sensor_Hub:Conn_JST_PH_2P -> Conn_JST_PH_2P
- U1: symbol Sensor_Hub:Raytac_MDBT50Q -> Raytac_MDBT50Q
- U2: symbol Sensor_Hub:Bosch_BME280 -> BME280
- U3: symbol Sensor_Hub:ST_LSM6DSO -> LSM6DSO
- U4: symbol Sensor_Hub:MCP73831T -> MCP73831T
- U5: symbol Sensor_Hub:TPS7A2033 -> TPS7A2033
Changed lines of the file:
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@@
 	)
 	(symbol
-		(lib_id "Sensor_Hub:Raytac_MDBT50Q")
+		(lib_id "Raytac_MDBT50Q")
 		(at 240 100 0)
 		(unit 1)
@@
 	)
 	(symbol
-		(lib_id "Sensor_Hub:Bosch_BME280")
+		(lib_id "BME280")
 		(at 330 70 0)
 		(unit 1)
@@
 	)
 	(symbol
-		(lib_id "Sensor_Hub:ST_LSM6DSO")
+		(lib_id "LSM6DSO")
 		(at 330 140 0)
 		(unit 1)
@@
 	)
 	(symbol
-		(lib_id "Sensor_Hub:MCP73831T")
+		(lib_id "MCP73831T")
 		(at 80 80 0)
 		(unit 1)
@@
 	)
 	(symbol
-		(lib_id "Sensor_Hub:TPS7A2033")
+		(lib_id "TPS7A2033")
 		(at 150 80 0)
 		(unit 1)
@@
 	)
 	(symbol
-		(lib_id "Sensor_Hub:SWD_Header_10Pin")
+		(lib_id "SWD_Header_10Pin")
 		(at 240 180 0)
 		(unit 1)
@@
 	)
 	(symbol
-		(lib_id "Sensor_Hub:USB_C_Receptacle_16P")
+		(lib_id "USB_C_Receptacle_16P")
 		(at 30 80 0)
 		(unit 1)
@@
 	)
 	(symbol
-		(lib_id "Sensor_Hub:Conn_JST_PH_2P")
+		(lib_id "Conn_JST_PH_2P")
 		(at 80 140 0)
 		(unit 1)
