File: hardware/nrf52840_sensor_hub.kicad_pcb (KiCad board)
At the start: 4 copper layers, 50 x 35 mm, 8 parts, among them J1 SWD_10P, J2 TYPE-C-16P, J3 JST-PH-2P, U1 Raytac MDBT50Q-1M, U2 BME280, U3 LSM6DSO, U4 MCP73831T, U5 TPS7A2033

Commit message: fix: programmatically generate KiCad 9 schema compliant project files
Other:
- board text added: "50mm x 35mm Sensor Hub (KiCad 8/9)"
- board text removed: "50mm x 35mm Sensor Hub (KiCad 8)"
Changed lines of the file:
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@@
 		(layer "Edge.Cuts")
 	)
-	(gr_text "50mm x 35mm Sensor Hub (KiCad 8)" (at 125 102.5)
+	(gr_text "50mm x 35mm Sensor Hub (KiCad 8/9)" (at 125 102.5)
 		(layer "F.SilkS")
 		(effects (font (size 0.9 0.9) (thickness 0.15)))
